Commit message: Make Husky even more multi-robot friendly.

File: husky_description/urdf/decorations.urdf.xacro (robot description, xacro)
@@ -8,9 +8,9 @@
   <material name="white"><color rgba="1.0 1.0 1.0 1.0" /></material>
   <material name="red"><color rgba="1.0 0.0 0.0 1.0" /></material>
-  <xacro:macro name="husky_decorate">
+  <xacro:macro name="husky_decorate" params="prefix" >
     <xacro:property name="husky_front_bumper_extend" value="$(optenv HUSKY_FRONT_BUMPER_EXTEND 0)" />
     <xacro:property name="husky_rear_bumper_extend" value="$(optenv HUSKY_REAR_BUMPER_EXTEND 0)" />
     <!-- Spawn Husky chassis -->
-    <link name="top_chassis_link">
+    <link name="${prefix}top_chassis_link">
       <visual>
         <origin xyz="0 0 0" rpy="0 0 0" />
@@ -21,11 +21,11 @@
     </link>
     <!-- Attach chassis to the robot -->
-    <joint name="top_chassis_joint" type="fixed">
-      <parent link="base_link" />
-      <child link="top_chassis_link" />
+    <joint name="${prefix}top_chassis_joint" type="fixed">
+      <parent link="${prefix}base_link" />
+      <child link="${prefix}top_chassis_link" />
     </joint>
     <xacro:if value="$(optenv HUSKY_USER_RAIL_ENABLED true)">
       <!-- Spawn user rails -->
-      <link name="user_rail_link">
+      <link name="${prefix}user_rail_link">
         <visual>
           <geometry>
@@ -35,12 +35,12 @@
       </link>
       <!-- Attach user rails to base link -->
-      <joint name="user_rail" type="fixed">
+      <joint name="${prefix}user_rail" type="fixed">
         <origin xyz="0.272 0 0.245" rpy="0 0 0" />
-        <parent link="base_link" />
-        <child link="user_rail_link" />
+        <parent link="${prefix}base_link" />
+        <child link="${prefix}user_rail_link" />
       </joint>
     </xacro:if>
     <!-- Spawn front bumper link -->
-    <link name="front_bumper_link">
+    <link name="${prefix}front_bumper_link">
       <visual>
         <geometry>
@@ -50,11 +50,11 @@
     </link>
     <!-- Attach front bumper -->
-    <joint name="front_bumper" type="fixed">
+    <joint name="${prefix}front_bumper" type="fixed">
       <origin xyz="${0.48 + husky_front_bumper_extend} 0 0.091" rpy="0 0 0" />
-      <parent link="base_link" />
-      <child link="front_bumper_link" />
+      <parent link="${prefix}base_link" />
+      <child link="${prefix}front_bumper_link" />
     </joint>
     <xacro:if value="${husky_front_bumper_extend}">
-      <link name="front_bumper_extension_link">
+      <link name="vfront_bumper_extension_link">
           <visual>
               <geometry>
@@ -63,12 +63,12 @@
           </visual>
       </link>
-      <joint name="front_bumper_extension" type="fixed">
+      <joint name="${prefix}front_bumper_extension" type="fixed">
         <origin xyz="${0.48 + husky_front_bumper_extend} 0 0.091" rpy="0 0 0" />
-        <parent link="base_link" />
-        <child link="front_bumper_extension_link" />
+        <parent link="${prefix}base_link" />
+        <child link="${prefix}front_bumper_extension_link" />
       </joint>
     </xacro:if>
     <!-- Spawn rear bumper link -->
-    <link name="rear_bumper_link">
+    <link name="${prefix}rear_bumper_link">
       <visual>
         <geometry>
@@ -78,11 +78,11 @@
     </link>
     <!-- Attach rear bumper -->
-    <joint name="rear_bumper" type="fixed">
+    <joint name="${prefix}rear_bumper" type="fixed">
       <origin xyz="${-0.48 - husky_rear_bumper_extend} 0 0.091" rpy="0 0 ${M_PI}" />
-      <parent link="base_link" />
-      <child link="rear_bumper_link" />
+      <parent link="${prefix}base_link" />
+      <child link="${prefix}rear_bumper_link" />
     </joint>
     <xacro:if value="${husky_rear_bumper_extend}">
-      <link name="rear_bumper_extension_link">
+      <link name="${prefix}rear_bumper_extension_link">
           <visual>
               <geometry>
@@ -91,8 +91,8 @@
           </visual>
       </link>
-      <joint name="rear_bumper_extension" type="fixed">
+      <joint name="${prefix}rear_bumper_extension" type="fixed">
         <origin xyz="${-0.48 - husky_rear_bumper_extend} 0 0.091" rpy="0 0 ${M_PI}" />
-        <parent link="base_link" />
-        <child link="rear_bumper_extension_link" />
+        <parent link="${prefix}base_link" />
+        <child link="${prefix}rear_bumper_extension_link" />
       </joint>
     </xacro:if>
@@ -100,5 +100,5 @@
       <!-- Spawn the top plate -->
       <xacro:if value="$(optenv HUSKY_LARGE_TOP_PLATE false)">
-        <link name="top_plate_link">
+        <link name="${prefix}top_plate_link">
           <visual>
             <origin xyz="0 0 0" rpy="0 0 0" />
@@ -115,18 +115,18 @@
         </link>
         <!-- Attach top plate -->
-        <joint name="top_plate_joint" type="fixed">
-          <parent link="base_link" />
-          <child link="top_plate_link"/>
+        <joint name="${prefix}top_plate_joint" type="fixed">
+          <parent link="${prefix}base_link" />
+          <child link="${prefix}top_plate_link"/>
           <origin xyz="0.0812 0 0.225" rpy="0 0 0"/>
         </joint>
         <!-- Top plate front link -->
-        <joint name="top_plate_front_joint" type="fixed">
-          <parent link="top_plate_link" />
-          <child link="top_plate_front_link"/>
+        <joint name="${prefix}top_plate_front_joint" type="fixed">
+          <parent link="${prefix}top_plate_link" />
+          <child link="${prefix}top_plate_front_link"/>
           <origin xyz="0.4125 0 0.00672" rpy="0 0 0"/>
         </joint>
         <!-- Top plate rear link-->
-        <joint name="top_plate_rear_joint" type="fixed">
-          <parent link="top_plate_link" />
+        <joint name="${prefix}top_plate_rear_joint" type="fixed">
+          <parent link="${prefix}top_plate_link" />
           <child link="top_plate_rear_link"/>
           <origin xyz="-0.4125 0 0.00672" rpy="0 0 0"/>
@@ -134,5 +134,5 @@
       </xacro:if>
       <xacro:unless value="$(optenv HUSKY_LARGE_TOP_PLATE false)">
-        <link name="top_plate_link">
+        <link name="${prefix}top_plate_link">
           <visual>
             <origin xyz="0 0 0" rpy="0 0 0" />
@@ -149,24 +149,24 @@
         </link>
         <!-- Attach top plate -->
-        <joint name="top_plate_joint" type="fixed">
-          <parent link="base_link" />
-          <child link="top_plate_link"/>
+        <joint name="${prefix}top_plate_joint" type="fixed">
+          <parent link="${prefix}base_link" />
+          <child link="${prefix}top_plate_link"/>
           <origin xyz="0.0812 0 0.245" rpy="0 0 0"/>
         </joint>
         <!-- Top plate front link -->
-        <joint name="top_plate_front_joint" type="fixed">
-          <parent link="top_plate_link" />
-          <child link="top_plate_front_link"/>
+        <joint name="${prefix}top_plate_front_joint" type="fixed">
+          <parent link="${prefix}top_plate_link" />
+          <child link="${prefix}top_plate_front_link"/>
           <origin xyz="0.36367 0 0.00639" rpy="0 0 0"/>
         </joint>
         <!-- Top plate rear link-->
-        <joint name="top_plate_rear_joint" type="fixed">
-          <parent link="top_plate_link" />
-          <child link="top_plate_rear_link"/>
+        <joint name="${prefix}top_plate_rear_joint" type="fixed">
+          <parent link="${prefix}top_plate_link" />
+          <child link="${prefix}top_plate_rear_link"/>
           <origin xyz="-0.36633 0 0.00639" rpy="0 0 0"/>
         </joint>
       </xacro:unless>
-      <link name="top_plate_front_link"/>
-      <link name="top_plate_rear_link"/>
+      <link name="${prefix}top_plate_front_link"/>
+      <link name="${prefix}top_plate_rear_link"/>
     </xacro:if>
   </xacro:macro>

File: husky_description/urdf/husky_macro.urdf.xacro (robot description, xacro)
@@ -89,17 +89,17 @@
     </joint>
     <!-- Husky wheel macros -->
-    <xacro:husky_wheel wheel_prefix="${prefix}front_left">
+    <xacro:husky_wheel prefix="${prefix}" wheel_prefix="front_left">
       <origin xyz="${wheelbase/2} ${track/2} ${wheel_vertical_offset}" rpy="0 0 0" />
     </xacro:husky_wheel>
-    <xacro:husky_wheel wheel_prefix="${prefix}front_right">
+    <xacro:husky_wheel prefix="${prefix}" wheel_prefix="front_right">
       <origin xyz="${wheelbase/2} ${-track/2} ${wheel_vertical_offset}" rpy="0 0 0" />
     </xacro:husky_wheel>
-    <xacro:husky_wheel wheel_prefix="${prefix}rear_left">
+    <xacro:husky_wheel prefix="${prefix}" wheel_prefix="rear_left">
       <origin xyz="${-wheelbase/2} ${track/2} ${wheel_vertical_offset}" rpy="0 0 0" />
     </xacro:husky_wheel>
-    <xacro:husky_wheel wheel_prefix="${prefix}rear_right">
+    <xacro:husky_wheel prefix="${prefix}" wheel_prefix="rear_right">
       <origin xyz="${-wheelbase/2} ${-track/2} ${wheel_vertical_offset}" rpy="0 0 0" />
     </xacro:husky_wheel>
-    <xacro:husky_decorate />
+    <xacro:husky_decorate prefix="${prefix}" />
     <!-- <xacro:if value="$(arg laser_enabled)">
       <xacro:sick_lms1xx_mount prefix="base"/>

File: husky_description/urdf/wheel.urdf.xacro (robot description, xacro)
@@ -1,6 +1,6 @@
 <?xml version="1.0"?>
 <robot xmlns:xacro="http://ros.org/wiki/xacro" name="husky_wheel">
-  <xacro:macro name="husky_wheel" params="wheel_prefix *joint_pose">
-    <link name="${wheel_prefix}_wheel">
+  <xacro:macro name="husky_wheel" params="prefix wheel_prefix *joint_pose">
+    <link name="${prefix}${wheel_prefix}_wheel">
       <inertial>
         <mass value="2.637" />
@@ -21,5 +21,5 @@
       </collision>
     </link>
-    <gazebo reference="${wheel_prefix}_wheel">
+    <gazebo reference="${prefix}${wheel_prefix}_wheel">
       <mu1 value="1.0"/>
       <mu2 value="0.5"/>
@@ -28,7 +28,7 @@
       <fdir1 value="1 0 0"/>
     </gazebo>
-    <joint name="${wheel_prefix}_wheel_joint" type="continuous">
-      <parent link="base_link"/>
-      <child link="${wheel_prefix}_wheel"/>
+    <joint name="${prefix}${wheel_prefix}_wheel_joint" type="continuous">
+      <parent link="${prefix}base_link"/>
+      <child link="${prefix}${wheel_prefix}_wheel"/>
       <xacro:insert_block name="joint_pose"/>
       <axis xyz="0 1 0" rpy="0 0 0" />
